File: 2024_PiezoPreamp3_Enclosure.kicad_pcb (KiCad board)
At the start: 2 copper layers, 83.5 x 81.6 mm, 9 parts

Commit message: working on the enclosure sides, edge cuts
Parts:
- removed the G*** at (192.3, 118.8)
- removed the G*** at (130.6, 133.5)
- removed TREBLE2: MountingHole_6mm_Pad, MountingHole:MountingHole_6mm_Pad
- added BACK: Board, PCM_kikit:Board, F.Cu at (178.2, 143.3)
- added BOTTOM2: Board, PCM_kikit:Board, F.Cu at (171.4, 190.9)
- added FRONT: Board, PCM_kikit:Board, F.Cu at (178.2, 93.6)
- added G***: LOGO, LOGO, F.Cu at (360.2, 115.0)
- added Hole: MountingHole_2.1mm, MountingHole:MountingHole_2.1mm, F.Cu at (238.3, 52.9)
- added Hole: MountingHole_2.1mm, MountingHole:MountingHole_2.1mm, F.Cu at (247.8, 76.8)
- added Hole: MountingHole_2.1mm, MountingHole:MountingHole_2.1mm, F.Cu at (247.8, 46.2)
- added Hole: MountingHole_2.1mm, MountingHole:MountingHole_2.1mm, F.Cu at (215.4, 78.0)
- added Hole: MountingHole_2.1mm, MountingHole:MountingHole_2.1mm, F.Cu at (247.8, 204.8)
- added Hole: MountingHole_2.1mm, MountingHole:MountingHole_2.1mm, F.Cu at (247.8, 235.4)
- added Hole: MountingHole_2.1mm, MountingHole:MountingHole_2.1mm, F.Cu at (215.4, 52.9)
- added Hole: MountingHole_2.1mm, MountingHole:MountingHole_2.1mm, F.Cu at (192.6, 52.9)
- added Hole: MountingHole_2.1mm, MountingHole:MountingHole_2.1mm, F.Cu at (183.1, 235.4)
- added Hole: MountingHole_2.1mm, MountingHole:MountingHole_2.1mm, F.Cu at (183.1, 76.8)
- added Hole: MountingHole_2.1mm, MountingHole:MountingHole_2.1mm, F.Cu at (183.1, 204.8)
- added Hole: MountingHole_2.1mm, MountingHole:MountingHole_2.1mm, F.Cu at (183.1, 46.2)
- moved G*** 156.8 mm to (358.9, 80.0)
- moved G*** 156.8 mm to (365.5, 95.8)
- moved G*** 133.1 mm to (335.3, 72.4)
- moved RIGHT 112.6 mm to (273.4, 93.6)
- moved TOP 75.3 mm to (176.2, 39.3)
- moved LEFT 38.6 mm to (123.5, 93.6)
Other:
- board size 83.5 x 81.6 mm -> 194.2 x 210.1 mm
- board text added: "Adult males shake tree branches during the mating season, effectively using vibrations to communicate."
- board text added: "Arx Piezo Preamp v3.0 2024/03"
- board text added: "BAXANDALL CENTER"
- board text added: "BOTTOM 1.6mm"
- board text added: "Embryos of the red-eyed tree frog detect vibrations of predators to hatch early and escape into the water."
- board text added: "HIGH-PASS FILTER"
- board text added: "ON"
- board text added: "PCB 1.6mm"
- board text added: "PIEZO GAIN"
- board text added: "PIEZO PREAMP"
- board text added: "TOP 1.6mm"
- board text added: "TRUE BYPASS"
- board text added: "bottom standoff 20mm"
- board text added: "silkscreen: white soldermask: black copper: silver/gold core: dirty white"
- board text added: "top standoff 15mm"
- board text added: "with frogs & trees"
- board text removed: "ASDF"

Commit message: working on text markings
Parts:
- moved BACK 11.3 mm to (178.2, 154.7)
- moved BOTTOM2 11.3 mm to (171.4, 202.2)
- moved Hole 11.3 mm to (247.8, 216.2)
- moved Hole 11.3 mm to (247.8, 246.8)
- moved Hole 11.3 mm to (183.1, 246.8)
- moved Hole 11.3 mm to (183.1, 216.2)
Other:
- board size 194.2 x 210.1 mm -> 194.2 x 221.3 mm
- board text added: "1k"
- board text added: "350"
- board text added: "600"
- board text added: "CENT"
- board text added: "CENTER"
- board text added: "GAIN"
- board text added: "HPF"
- board text added: "TONE CENTER"
- board text added: "▲"
- board text removed: "BAXANDALL CENTER"
